Commit message: Create 2WD robot and create its gazebo sim, slam.

File: src/warehouse_robot_description/urdf/4wd_warehouse_robots.urdf.xacro (robot description, xacro)
@@ -35,5 +35,5 @@
       <origin xyz="0 0 0" rpy="0 0 0"/>
       <geometry>
-        <mesh filename="package://warehouse_robot_description/meshes/base_link.STL"
+        <mesh filename="package://warehouse_robot_description/meshes/4wd/base_link.STL"
               scale="${S} ${S} ${S}"/>
       </geometry>
@@ -43,5 +43,5 @@
       <origin xyz="0 0 0" rpy="0 0 0"/>
       <geometry>
-        <mesh filename="package://warehouse_robot_description/meshes/base_link.STL"
+        <mesh filename="package://warehouse_robot_description/meshes/4wd/base_link.STL"
               scale="${S} ${S} ${S}"/>
       </geometry>
@@ -66,5 +66,5 @@
         <origin xyz="0 0 0" rpy="0 0 0"/>
         <geometry>
-          <mesh filename="package://warehouse_robot_description/meshes/${mesh}"
+          <mesh filename="package://warehouse_robot_description/meshes/4wd/${mesh}"
                 scale="${S} ${S} ${S}"/>
         </geometry>
@@ -74,5 +74,5 @@
         <origin xyz="0 0 0" rpy="0 0 0"/>
         <geometry>
-          <mesh filename="package://warehouse_robot_description/meshes/${mesh}"
+          <mesh filename="package://warehouse_robot_description/meshes/4wd/${mesh}"
                 scale="${S} ${S} ${S}"/>
         </geometry>
