Commit message: Update multirobot.launch.py and its dependencies

File: src/warehouse_robot_description/urdf/2wd_multirobot.urdf.xacro (robot description, xacro)
@@ -1,11 +1,13 @@
 <?xml version="1.0" encoding="utf-8"?>
 <robot xmlns:xacro="http://www.ros.org/wiki/xacro" name="2wd_warehouse_robot">
+  <xacro:arg name="prefix" default="" />
+  <xacro:arg name="robot_name" default="warehouse_bot" />
   <!-- ===========================
        base_footprint
   ============================ -->
-  <link name="base_footprint"/>
-  <joint name="base_joint" type="fixed">
-    <parent link="base_footprint"/>
-    <child link="base_link"/>
+  <link name="$(arg prefix)base_footprint"/>
+  <joint name="$(arg prefix)base_joint" type="fixed">
+    <parent link="$(arg prefix)base_footprint"/>
+    <child link="$(arg prefix)base_link"/>
     <origin xyz="0 0 0" rpy="0 0 0"/>
   </joint>
@@ -13,5 +15,5 @@
        Base link
   ============================ -->
-  <link name="base_link">
+  <link name="$(arg prefix)base_link">
     <inertial>
       <!-- Reduced mass for simulation stability (Original ~305kg -> Scaled to ~30kg) -->
@@ -42,5 +44,5 @@
   ============================ -->
   <!-- Left Wheel -->
-  <link name="left_wheel">
+  <link name="$(arg prefix)left_wheel">
     <inertial>
       <origin xyz="0 0 0.033" rpy="0 0 0" />
@@ -65,13 +67,13 @@
     </collision>
   </link>
-  <joint name="left_wheel_joint" type="continuous">
+  <joint name="$(arg prefix)left_wheel_joint" type="continuous">
     <origin xyz="-0.48569 0.55575 -0.1755" rpy="1.5708 0 0" />
-    <parent link="base_link" />
-    <child link="left_wheel" />
+    <parent link="$(arg prefix)base_link" />
+    <child link="$(arg prefix)left_wheel" />
     <axis xyz="0 0 -1" />
     <limit effort="100" velocity="10" />
   </joint>
   <!-- Right Wheel -->
-  <link name="right_wheel">
+  <link name="$(arg prefix)right_wheel">
     <inertial>
       <origin xyz="0 0 -0.033" rpy="0 0 0" />
@@ -96,8 +98,8 @@
     </collision>
   </link>
-  <joint name="right_wheel_joint" type="continuous">
+  <joint name="$(arg prefix)right_wheel_joint" type="continuous">
     <origin xyz="-0.48569 -0.55575 -0.1755" rpy="1.5708 0 0" />
-    <parent link="base_link" />
-    <child link="right_wheel" />
+    <parent link="$(arg prefix)base_link" />
+    <child link="$(arg prefix)right_wheel" />
     <axis xyz="0 0 -1" />
     <limit effort="100" velocity="10" />
@@ -106,5 +108,5 @@
        Caster Wheel Assembly
   ============================ -->
-  <link name="caster_connection">
+  <link name="$(arg prefix)caster_connection">
     <inertial>
       <origin xyz="-0.03 0 -0.11" rpy="0 0 0" />
@@ -128,11 +130,11 @@
     </collision>
   </link>
-  <joint name="caster_connection_joint" type="continuous">
+  <joint name="$(arg prefix)caster_connection_joint" type="continuous">
     <origin xyz="0.50656 0 0" rpy="0 0 0" />
-    <parent link="base_link" />
-    <child link="caster_connection" />
+    <parent link="$(arg prefix)base_link" />
+    <child link="$(arg prefix)caster_connection" />
     <axis xyz="0 0 -1" />
   </joint>
-  <link name="caster_wheel">
+  <link name="$(arg prefix)caster_wheel">
     <inertial>
       <origin xyz="0 0 0" rpy="0 0 0" />
@@ -156,12 +158,12 @@
     </collision>
   </link>
-  <joint name="caster_wheel_joint" type="continuous">
+  <joint name="$(arg prefix)caster_wheel_joint" type="continuous">
     <origin xyz="-0.13927 -0.0053 -0.22785" rpy="1.5708 0 0" />
-    <parent link="caster_connection" />
-    <child link="caster_wheel" />
+    <parent link="$(arg prefix)caster_connection" />
+    <child link="$(arg prefix)caster_wheel" />
     <axis xyz="0 0 1" />
   </joint>
   <!-- Frictionless Caster (Critical for smooth turning) -->
-  <gazebo reference="caster_wheel">
+  <gazebo reference="$(arg prefix)caster_wheel">
     <mu1>200.0</mu1>
     <mu2>100.0</mu2>
@@ -169,5 +171,5 @@
     <kd>1.0</kd>
   </gazebo>
-  <gazebo reference="caster_connection">
+  <gazebo reference="$(arg prefix)caster_connection">
     <mu1>200.0</mu1>
     <mu2>100.0</mu2>
@@ -178,5 +180,5 @@
        Sensor (LiDAR)
   ============================ -->
- <link name="lidar_link">
+ <link name="$(arg prefix)lidar_link">
     <inertial>
       <origin xyz="-0.0466543100833166 7.97140131680862E-14 0.119806074995455" rpy="0 0 0" />
@@ -202,19 +204,19 @@
   </link>
   <joint
-    name="lidar_joint"
+    name="$(arg prefix)lidar_joint"
     type="fixed">
     <origin xyz="0.50656 0 0.42188" rpy="3.1416 0 0" />
-    <parent link="base_link" />
-    <child link="lidar_link" />
+    <parent link="$(arg prefix)base_link" />
+    <child link="$(arg prefix)lidar_link" />
     <axis xyz="0 0 0" />
   </joint>
-  <gazebo reference="lidar_link">
-    <sensor name="lidar" type="gpu_lidar">
+  <gazebo reference="$(arg prefix)lidar_link">
+    <sensor name="lidar" type="lidar">
       <always_on>true</always_on>
       <visualize>true</visualize>
       <topic>scan</topic>
       <update_rate>50</update_rate>
-      <gz_frame_id>lidar_link</gz_frame_id>
-      <frame_id>lidar_link</frame_id>
+      <gz_frame_id>$(arg prefix)lidar_link</gz_frame_id>
+      <frame_id>$(arg prefix)lidar_link</frame_id>
       <ray>
         <scan>
@@ -237,9 +239,9 @@
     </sensor>
   </gazebo>
-  <gazebo reference="lidar_link">
+  <gazebo reference="$(arg prefix)lidar_link">
     <plugin filename="ignition-gazebo-pose-publisher-system.so"
             name="ignition::gazebo::systems::PosePublisher">
       <publish_tf>true</publish_tf>
-      <frame_id>lidar_link</frame_id>
+      <frame_id>$(arg prefix)lidar_link</frame_id>
     </plugin>
   </gazebo>
@@ -251,6 +253,6 @@
             name="ignition::gazebo::systems::DiffDrive">
       <!-- Joints -->
-      <left_joint>left_wheel_joint</left_joint>
-      <right_joint>right_wheel_joint</right_joint>
+      <left_joint>$(arg prefix)left_wheel_joint</left_joint>
+      <right_joint>$(arg prefix)right_wheel_joint</right_joint>
       <!-- <wheel_separation>1.1115</wheel_separation> -->
       <wheel_separation>0.8</wheel_separation>
@@ -259,9 +261,9 @@
       <max_acceleration>10</max_acceleration>
       <!-- Topics -->
-      <topic>/cmd_vel</topic>
-      <odom_topic>/odom</odom_topic>
-      <tf_topic>/tf</tf_topic>
-      <frame_id>odom</frame_id>
-      <child_frame_id>base_footprint</child_frame_id>
+      <topic>/model/$(arg robot_name)/cmd_vel</topic>
+      <odom_topic>/model/$(arg robot_name)/odom</odom_topic>
+      <tf_topic>/model/$(arg robot_name)/tf</tf_topic>
+      <frame_id>$(arg prefix)odom</frame_id>
+      <child_frame_id>$(arg prefix)base_footprint</child_frame_id>
       <odom_publish_frequency>50</odom_publish_frequency>
     </plugin>
@@ -273,5 +275,5 @@
   <plugin filename="libignition-gazebo-joint-state-publisher-system.so"
           name="ignition::gazebo::systems::JointStatePublisher">
-    <topic>joint_states</topic>
+    <topic>/model/$(arg robot_name)/joint_states</topic>
   </plugin>
   </gazebo>
